Commit message: hello

File: robobase_description/models/bases/rectangular-base.urdf.xacro (robot description, xacro)
@@ -17,13 +17,7 @@
     <origin xyz="0 0 0" rpy="0 0 0"/>
 </joint>
+<!-- Compute base mass -->
 <link name="base_link">
-    <xacro:cuboid_inertia x="${base_length}" y="${base_width}" z="${base_height}" prefix="base"/>
-    <inertial>
-        <mass value="${base_mass}"/>
-        <inertia
-            ixx="${base_ixx}" ixy="0" ixz="0"
-            iyy="${base_iyy}" iyz="0"
-            izz="${base_izz}"/>
-    </inertial>
+    <xacro:inertial_box x="${base_length}" y="${base_width}" z="${base_height}"/>
     <visual>
         <origin xyz="0 0 ${base_height / 2}" rpy="0 0 0"/>
@@ -49,13 +43,7 @@
     <axis xyz="0 0 1"/>
 </joint>
+<!-- Compute wheel mass -->
 <link name="lfwheel_link">
-    <xacro:cylinder_inertia radius="${wheel_radius}" length="${wheel_width}" prefix="lfwheel"/>
-    <inertial>
-        <mass value="${wheel_mass}"/>
-        <inertia
-            ixx="${lfwheel_ixx}" ixy="0" ixz="0"
-            iyy="${lfwheel_iyy}" iyz="0"
-            izz="${lfwheel_izz}"/>
-    </inertial>
+    <xacro:inertial_cylinder radius="${wheel_radius}" length="${wheel_width}"/>
     <visual>
         <origin xyz="0 0 ${wheel_width / 2}" rpy="0 0 0"/>
@@ -74,3 +62,3 @@
     </collision>
 </link>
-<robot name="mobile_base">
+</robot>

File: robobase_description/models/inertia_macros.xacro (robot description, xacro)
@@ -1,30 +1,40 @@
 <robot xmlns:xacro="http://ros.org/wiki/xacro">
-  <!-- Default density in kg/m^3 (e.g., aluminum ~2700) -->
+  <!-- Default density (kg/m^3) -->
   <xacro:property name="default_density" value="2700"/>
-  <xacro:macro name="cylinder_inertia" params="radius length mass:=None density:=${default_density} prefix:=cyl">
-    <!-- Calculate mass if not provided -->
-    <xacro:if value="${mass == 'None'}">
-      <xacro:property name="${prefix}_mass" value="${density * 3.14159265359 * radius * radius * length}"/>
+  <!-- Inertial for a box (URDF axes aligned, origin at box center) -->
+  <!-- If mass not provided, computed as density * x * y * z -->
+  <xacro:macro name="inertial_box" params="x y z mass:='' density:=${default_density} *origin">
+    <xacro:if value="${mass == ''}">
+      <xacro:property name="_ibox_mass" value="${density * x * y * z}"/>
     </xacro:if>
-    <xacro:if value="${mass != 'None'}">
-      <xacro:property name="${prefix}_mass" value="${mass}"/>
+    <xacro:if value="${mass != ''}">
+      <xacro:property name="_ibox_mass" value="${mass}"/>
     </xacro:if>
-    <!-- Inertia about center (z axis is cylinder axis) -->
-    <xacro:property name="${prefix}_ixx" value="${0.5 * ${prefix}_mass * radius * radius}"/>
-    <xacro:property name="${prefix}_iyy" value="${0.5 * ${prefix}_mass * radius * radius}"/>
-    <xacro:property name="${prefix}_izz" value="${(1/12.0) * ${prefix}_mass * (3 * radius * radius + length * length)}"/>
+    <inertial>
+      <xacro:insert_block name="origin"/>
+      <mass value="${_ibox_mass}"/>
+      <inertia
+        ixx="${(1/12.0) * _ibox_mass * (y*y + z*z)}" ixy="0" ixz="0"
+        iyy="${(1/12.0) * _ibox_mass * (x*x + z*z)}" iyz="0"
+        izz="${(1/12.0) * _ibox_mass * (x*x + y*y)}"/>
+    </inertial>
   </xacro:macro>
-  <xacro:macro name="cuboid_inertia" params="x y z mass:=None density:=${default_density} prefix:=cub">
-    <!-- Calculate mass if not provided -->
-    <xacro:if value="${mass == 'None'}">
-      <xacro:property name="${prefix}_mass" value="${density * x * y * z}"/>
+  <!-- Inertial for a solid cylinder whose axis is the URDF Z axis -->
+  <!-- If mass not provided, computed as density * pi * r^2 * length -->
+  <xacro:macro name="inertial_cylinder" params="radius length mass:='' density:=${default_density} *origin">
+    <xacro:if value="${mass == ''}">
+      <xacro:property name="_icyl_mass" value="${density * 3.141592653589793 * radius * radius * length}"/>
     </xacro:if>
-    <xacro:if value="${mass != 'None'}">
-      <xacro:property name="${prefix}_mass" value="${mass}"/>
+    <xacro:if value="${mass != ''}">
+      <xacro:property name="_icyl_mass" value="${mass}"/>
     </xacro:if>
-    <!-- Inertia about center -->
-    <xacro:property name="${prefix}_ixx" value="${(1/12.0) * ${prefix}_mass * (y*y + z*z)}"/>
-    <xacro:property name="${prefix}_iyy" value="${(1/12.0) * ${prefix}_mass * (x*x + z*z)}"/>
-    <xacro:property name="${prefix}_izz" value="${(1/12.0) * ${prefix}_mass * (x*x + y*y)}"/>
+    <inertial>
+      <xacro:insert_block name="origin"/>
+      <mass value="${_icyl_mass}"/>
+      <inertia
+        ixx="${(1/12.0) * _icyl_mass * (3*radius*radius + length*length)}" ixy="0" ixz="0"
+        iyy="${(1/12.0) * _icyl_mass * (3*radius*radius + length*length)}" iyz="0"
+        izz="${0.5 * _icyl_mass * radius * radius}"/>
+    </inertial>
   </xacro:macro>
 </robot>

Commit message: hello

File: robobase_description/models/bases/rectangular-base.urdf.xacro (robot description, xacro)
@@ -19,5 +19,7 @@
 <!-- Compute base mass -->
 <link name="base_link">
-    <xacro:inertial_box x="${base_length}" y="${base_width}" z="${base_height}"/>
+    <xacro:inertial_box x="${base_length}" y="${base_width}" z="${base_height}">
+        <origin xyz="0 0 ${base_height / 2}" rpy="0 0 0"/>
+    </xacro:inertial_box>
     <visual>
         <origin xyz="0 0 ${base_height / 2}" rpy="0 0 0"/>
@@ -45,5 +47,7 @@
 <!-- Compute wheel mass -->
 <link name="lfwheel_link">
-    <xacro:inertial_cylinder radius="${wheel_radius}" length="${wheel_width}"/>
+    <xacro:inertial_cylinder radius="${wheel_radius}" length="${wheel_width}">
+        <origin xyz="0 0 ${wheel_width / 2}" rpy="0 0 0"/>
+    </xacro:inertial_cylinder>
     <visual>
         <origin xyz="0 0 ${wheel_width / 2}" rpy="0 0 0"/>

Commit message: hello

File: robobase_description/models/bases/rectangular-base.urdf.xacro (robot description, xacro)
@@ -5,7 +5,7 @@
 <xacro:property name="base_length" default="1"/>
 <xacro:property name="base_width" default="0.6"/>
-<xacro:property name="base_height" default="0.2"/>
-<xacro:property name="wheel_radius" default="0.2"/>
-<xacro:property name="wheel_width" default="0.1"/>
+<xacro:property name="base_height" default="0.3"/>
+<xacro:property name="wheel_radius" default="0.3"/>
+<xacro:property name="wheel_width" default="0.25"/>
 <link name="base_footprint">
     <origin xyz="0 0 0" rpy="0 0 0"/>
@@ -17,5 +17,4 @@
     <origin xyz="0 0 0" rpy="0 0 0"/>
 </joint>
-<!-- Compute base mass -->
 <link name="base_link">
     <xacro:inertial_box x="${base_length}" y="${base_width}" z="${base_height}">
@@ -45,5 +44,4 @@
     <axis xyz="0 0 1"/>
 </joint>
-<!-- Compute wheel mass -->
 <link name="lfwheel_link">
     <xacro:inertial_cylinder radius="${wheel_radius}" length="${wheel_width}">
@@ -66,3 +64,84 @@
     </collision>
 </link>
+<!-- Rfwheel Link -->
+<joint name="rfwheel_joint" type="continuous">
+    <parent link="base_link"/>
+    <child link="rfwheel_link"/>
+    <origin xyz="${base_length / 2} -${base_width / 2} ${base_height / 2}" rpy="${pi / 2} 0 0"/>
+    <axis xyz="0 0 -1"/>
+</joint>
+<link name="rfwheel_link">
+    <xacro:inertial_cylinder radius="${wheel_radius}" length="${wheel_width}">
+        <origin xyz="0 0 ${wheel_width / 2}" rpy="0 0 0"/>
+    </xacro:inertial_cylinder>
+    <visual>
+        <origin xyz="0 0 ${wheel_width / 2}" rpy="0 0 0"/>
+        <geometry>
+            <cylinder radius="${wheel_radius}" length="${wheel_width}"/>
+        </geometry>
+        <material name="black">
+            <xacro:black/>
+        </material>
+    </visual>
+    <collision>
+        <origin xyz="0 0 ${wheel_width / 2}" rpy="0 0 0"/>
+        <geometry>
+            <cylinder radius="${wheel_radius}" length="${wheel_width}"/>
+        </geometry>
+    </collision>
+</link>
+<!-- Lbwheel Link -->
+<joint name="lbwheel_joint" type="continuous">
+    <parent link="base_link"/>
+    <child link="lbwheel_link"/>
+    <origin xyz="-${base_length / 2} ${base_width / 2} ${base_height / 2}" rpy="-${pi / 2} 0 0"/>
+    <axis xyz="0 0 1"/>
+</joint>
+<link name="lbwheel_link">
+    <xacro:inertial_cylinder radius="${wheel_radius}" length="${wheel_width}">
+        <origin xyz="0 0 ${wheel_width / 2}" rpy="0 0 0"/>
+    </xacro:inertial_cylinder>
+    <visual>
+        <origin xyz="0 0 ${wheel_width / 2}" rpy="0 0 0"/>
+        <geometry>
+            <cylinder radius="${wheel_radius}" length="${wheel_width}"/>
+        </geometry>
+        <material name="black">
+            <xacro:black/>
+        </material>
+    </visual>
+    <collision>
+        <origin xyz="0 0 ${wheel_width / 2}" rpy="0 0 0"/>
+        <geometry>
+            <cylinder radius="${wheel_radius}" length="${wheel_width}"/>
+        </geometry>
+    </collision>
+</link>
+<!-- Rbwheel Link -->
+<joint name="rbwheel_joint" type="continuous">
+    <parent link="base_link"/>
+    <child link="rbwheel_link"/>
+    <origin xyz="-${base_length / 2} -${base_width / 2} ${base_height / 2}" rpy="${pi / 2} 0 0"/>
+    <axis xyz="0 0 -1"/>
+</joint>
+<link name="rbwheel_link">
+    <xacro:inertial_cylinder radius="${wheel_radius}" length="${wheel_width}">
+        <origin xyz="0 0 ${wheel_width / 2}" rpy="0 0 0"/>
+    </xacro:inertial_cylinder>
+    <visual>
+        <origin xyz="0 0 ${wheel_width / 2}" rpy="0 0 0"/>
+        <geometry>
+            <cylinder radius="${wheel_radius}" length="${wheel_width}"/>
+        </geometry>
+        <material name="black">
+            <xacro:black/>
+        </material>
+    </visual>
+    <collision>
+        <origin xyz="0 0 ${wheel_width / 2}" rpy="0 0 0"/>
+        <geometry>
+            <cylinder radius="${wheel_radius}" length="${wheel_width}"/>
+        </geometry>
+    </collision>
+</link>
 </robot>

Commit message: hello

File: robobase_description/models/bases/rectangular-base.urdf.xacro (robot description, xacro)
@@ -3,9 +3,4 @@
 <xacro:include filename="$(find robobase_description)/models/materials.urdf.xacro"/>
 <xacro:include filename="$(find robobase_description)/models/inertia_macros.xacro"/>
-<xacro:property name="base_length" default="1"/>
-<xacro:property name="base_width" default="0.6"/>
-<xacro:property name="base_height" default="0.3"/>
-<xacro:property name="wheel_radius" default="0.3"/>
-<xacro:property name="wheel_width" default="0.25"/>
 <link name="base_footprint">
     <origin xyz="0 0 0" rpy="0 0 0"/>

File: robobase_description/models/robo.urdf.xacro (robot description, xacro)
@@ -1,4 +1,10 @@
 <?xml version="1.0"?>
 <robot xmlns:xacro="http://www.ros.org/wiki/xacro" name="robobase">
+<xacro:property name="base_length" default="0.6"/>
+<xacro:property name="base_width" default="0.6"/>
+<xacro:property name="base_height" default="0.3"/>
+<xacro:property name="wheel_radius" default="0.3"/>
+<xacro:property name="wheel_width" default="0.25"/>
 <xacro:include filename="$(find robobase_description)/models/bases/rectangular-base.urdf.xacro"/>
+<xacro:include filename="$(find robobase_description)/models/sensors/camera.urdf.xacro"/>
 </robot>

Commit message: hello

File: robobase_description/models/bases/rectangular-base.urdf.xacro (robot description, xacro)
@@ -57,25 +57,12 @@
             <cylinder radius="${wheel_radius}" length="${wheel_width}"/>
         </geometry>
-        <surface>
-          <friction>
-            <ode>
-              <mu>0.2</mu>        <!-- Even lower -->
-              <mu2>0.1</mu2>      <!-- Very low lateral friction -->
-              <!-- <fdir1>1 0 0</fdir1> -->
-              <slip1>0.3</slip1>  <!-- Higher slip -->
-              <slip2>0.4</slip2>  <!-- Much higher lateral slip -->
-            </ode>
-          </friction>
-          <contact>
-            <ode>
-              <kp>1e6</kp>
-              <kd>1e4</kd>
-              <max_vel>0.2</max_vel>
-              <min_depth>0.001</min_depth>
-            </ode>
-          </contact>
-        </surface>
     </collision>
 </link>
+<gazebo reference="lfwheel_link">
+  <material>Gazebo/Black</material>
+  <kp>1e15</kp>
+  <kd>1e14</kd>
+  <fdir1>0 0 1</fdir1>
+</gazebo>
 <!-- Rfwheel Link -->
 <joint name="rfwheel_joint" type="continuous">
@@ -103,25 +90,12 @@
             <cylinder radius="${wheel_radius}" length="${wheel_width}"/>
         </geometry>
-        <surface>
-          <friction>
-            <ode>
-              <mu>0.2</mu>        <!-- Even lower -->
-              <mu2>0.1</mu2>      <!-- Very low lateral friction -->
-              <!-- <fdir1>1 0 0</fdir1> -->
-              <slip1>0.3</slip1>  <!-- Higher slip -->
-              <slip2>0.4</slip2>  <!-- Much higher lateral slip -->
-            </ode>
-          </friction>
-          <contact>
-            <ode>
-              <kp>1e6</kp>
-              <kd>1e4</kd>
-              <max_vel>0.2</max_vel>
-              <min_depth>0.001</min_depth>
-            </ode>
-          </contact>
-        </surface>
     </collision>
 </link>
+<gazebo reference="rfwheel_link">
+  <material>Gazebo/Black</material>
+  <kp>1e15</kp>
+  <kd>1e14</kd>
+  <fdir1>0 0 1</fdir1>
+</gazebo>
 <!-- Lbwheel Link -->
 <joint name="lbwheel_joint" type="continuous">
@@ -149,25 +123,12 @@
             <cylinder radius="${wheel_radius}" length="${wheel_width}"/>
         </geometry>
-        <surface>
-          <friction>
-            <ode>
-              <mu>0.2</mu>        <!-- Even lower -->
-              <mu2>0.1</mu2>      <!-- Very low lateral friction -->
-              <!-- <fdir1>1 0 0</fdir1> -->
-              <slip1>0.3</slip1>  <!-- Higher slip -->
-              <slip2>0.4</slip2>  <!-- Much higher lateral slip -->
-            </ode>
-          </friction>
-          <contact>
-            <ode>
-              <kp>1e6</kp>
-              <kd>1e4</kd>
-              <max_vel>0.2</max_vel>
-              <min_depth>0.001</min_depth>
-            </ode>
-          </contact>
-        </surface>
     </collision>
 </link>
+<gazebo reference="lbwheel_link">
+  <material>Gazebo/Black</material>
+  <kp>1e15</kp>
+  <kd>1e14</kd>
+  <fdir1>0 0 1</fdir1>
+</gazebo>
 <!-- Rbwheel Link -->
 <joint name="rbwheel_joint" type="continuous">
@@ -195,25 +156,12 @@
             <cylinder radius="${wheel_radius}" length="${wheel_width}"/>
         </geometry>
-        <surface>
-          <friction>
-            <ode>
-              <mu>0.2</mu>        <!-- Even lower -->
-              <mu2>0.1</mu2>      <!-- Very low lateral friction -->
-              <!-- <fdir1>1 0 0</fdir1> -->
-              <slip1>0.3</slip1>  <!-- Higher slip -->
-              <slip2>0.4</slip2>  <!-- Much higher lateral slip -->
-            </ode>
-          </friction>
-          <contact>
-            <ode>
-              <kp>1e6</kp>
-              <kd>1e4</kd>
-              <max_vel>0.2</max_vel>
-              <min_depth>0.001</min_depth>
-            </ode>
-          </contact>
-        </surface>
     </collision>
 </link>
+<gazebo reference="rbwheel_link">
+  <material>Gazebo/Black</material>
+  <kp>1e15</kp>
+  <kd>1e14</kd>
+  <fdir1>0 0 1</fdir1>
+</gazebo>
 <gazebo>
     <plugin name="gz::sim::systems::JointStatePublisher"

File: robobase_description/models/gazebo/4differential-drive.urdf.xacro (robot description, xacro)
@@ -13,5 +13,5 @@
     <right_joint>rfwheel_joint</right_joint>
     <right_joint>rbwheel_joint</right_joint>
-    <wheel_separation>0.525</wheel_separation>
+    <wheel_separation>0.6</wheel_separation>
       <wheel_radius>0.15</wheel_radius>
       <max_wheel_torque>500.0</max_wheel_torque>     <!-- Increase from default -->

Commit message: hello

File: robobase_description/models/bases/rectangular-base.urdf.xacro (robot description, xacro)
@@ -38,4 +38,6 @@
     <origin xyz="${base_length / 2} ${base_width / 2} ${base_height / 2}" rpy="-${pi / 2} 0 0"/>
     <axis xyz="0 0 1"/>
+    <limit effort="1000" velocity="1000"/>
+    <dynamics damping="1.0" friction="1.0"/>
 </joint>
 <link name="lfwheel_link">
@@ -60,10 +62,7 @@
 </link>
 <gazebo reference="lfwheel_link">
-  <material>Gazebo/Black</material>
-  <kp>1e15</kp>
-  <kd>1e14</kd>
-  <fdir1>0 0 1</fdir1>
-  <mu>1</mu>
-  <mu2>1</mu2>
+  <mu1>1.0</mu1>
+  <mu2>1.0</mu2>
+  <material>Gazebo/Yellow</material>
 </gazebo>
 <!-- Rfwheel Link -->
@@ -73,4 +72,6 @@
     <origin xyz="${base_length / 2} -${base_width / 2} ${base_height / 2}" rpy="${pi / 2} 0 0"/>
     <axis xyz="0 0 -1"/>
+    <limit effort="1000" velocity="1000"/>
+    <dynamics damping="1.0" friction="1.0"/>
 </joint>
 <link name="rfwheel_link">
@@ -95,10 +96,7 @@
 </link>
 <gazebo reference="rfwheel_link">
-  <material>Gazebo/Black</material>
-  <kp>1e15</kp>
-  <kd>1e14</kd>
-  <fdir1>0 0 1</fdir1>
-  <mu>1</mu>
-  <mu2>1</mu2>
+  <mu1>1.0</mu1>
+  <mu2>1.0</mu2>
+  <material>Gazebo/Yellow</material>
 </gazebo>
 <!-- Lbwheel Link -->
@@ -108,4 +106,6 @@
     <origin xyz="-${base_length / 2} ${base_width / 2} ${base_height / 2}" rpy="-${pi / 2} 0 0"/>
     <axis xyz="0 0 1"/>
+    <limit effort="1000" velocity="1000"/>
+    <dynamics damping="1.0" friction="1.0"/>
 </joint>
 <link name="lbwheel_link">
@@ -130,10 +130,7 @@
 </link>
 <gazebo reference="lbwheel_link">
-  <material>Gazebo/Black</material>
-  <kp>1e15</kp>
-  <kd>1e14</kd>
-  <fdir1>0 0 1</fdir1>
-  <mu>1</mu>
-  <mu2>1</mu2>
+  <mu1>1.0</mu1>
+  <mu2>1.0</mu2>
+  <material>Gazebo/Yellow</material>
 </gazebo>
 <!-- Rbwheel Link -->
@@ -143,4 +140,6 @@
     <origin xyz="-${base_length / 2} -${base_width / 2} ${base_height / 2}" rpy="${pi / 2} 0 0"/>
     <axis xyz="0 0 -1"/>
+    <limit effort="1000" velocity="1000"/>
+    <dynamics damping="1.0" friction="1.0"/>
 </joint>
 <link name="rbwheel_link">
@@ -165,10 +164,7 @@
 </link>
 <gazebo reference="rbwheel_link">
-  <material>Gazebo/Black</material>
-  <kp>1e15</kp>
-  <kd>1e14</kd>
-  <fdir1>0 0 1</fdir1>
-  <mu>1</mu>
-  <mu2>1</mu2>
+  <mu1>1.0</mu1>
+  <mu2>1.0</mu2>
+  <material>Gazebo/Yellow</material>
 </gazebo>
 <gazebo>

File: robobase_description/models/gazebo/4differential-drive.urdf.xacro (robot description, xacro)
@@ -14,5 +14,5 @@
     <right_joint>rbwheel_joint</right_joint>
     <wheel_separation>0.6</wheel_separation>
-      <wheel_radius>0.15</wheel_radius>
+    <wheel_diameter>0.3</wheel_diameter>
       <max_wheel_torque>500.0</max_wheel_torque>
       <max_linear_acceleration>5.0</max_linear_acceleration>

File: robobase_description/models/sensors/lidar.urdf.xacro (robot description, xacro)
@@ -48,5 +48,5 @@
           <range>
             <min>0.120000</min>
-            <max>4</max>
+            <max>8</max>
             <resolution>0.015000</resolution>
           </range>
