Commit message: hello

File: robobase_description/models/bases/rectangular-base.urdf.xacro (robot description, xacro)
@@ -36,17 +36,14 @@
     <parent link="base_link"/>
     <child link="lfwheel_link"/>
-    <origin xyz="${base_length / 2} ${base_width / 2} ${base_height / 2}" rpy="-${pi / 2} 0 0"/>
-    <axis xyz="0 0 1"/>
-    <limit effort="1000" velocity="1000"/>
-    <dynamics damping="1.0" friction="1.0"/>
+    <origin xyz="${base_length / 2} ${base_width / 2} 0" rpy="0 0 0"/>
 </joint>
 <link name="lfwheel_link">
-    <xacro:inertial_cylinder radius="${wheel_radius}" length="${wheel_width}">
-        <origin xyz="0 0 ${wheel_width / 2}" rpy="0 0 0"/>
-    </xacro:inertial_cylinder>
+    <xacro:inertial_sphere radius="${castor_radius}">
+        <origin xyz="0 0 0" rpy="0 0 0"/>
+    </xacro:inertial_sphere>
     <visual>
-        <origin xyz="0 0 ${wheel_width / 2}" rpy="0 0 0"/>
+        <origin xyz="0 0 0" rpy="0 0 0"/>
         <geometry>
-            <cylinder radius="${wheel_radius}" length="${wheel_width}"/>
+            <sphere radius="${castor_radius}"/>
         </geometry>
         <material name="black">
@@ -55,14 +52,18 @@
     </visual>
     <collision>
-        <origin xyz="0 0 ${wheel_width / 2}" rpy="0 0 0"/>
+        <origin xyz="0 0 0" rpy="0 0 0"/>
         <geometry>
-            <cylinder radius="${wheel_radius}" length="${wheel_width}"/>
+            <sphere radius="${castor_radius}"/>
         </geometry>
     </collision>
 </link>
 <gazebo reference="lfwheel_link">
+  <joint name="lfwheel_joint" type="ball">
+    <parent>base_link</parent>
+    <child>lfwheel_joint</child>
+  </joint>
   <mu1>1.0</mu1>
   <mu2>1.0</mu2>
-  <material>Gazebo/Yellow</material>
+  <material>Gazebo/Black</material>
 </gazebo>
 <!-- Rfwheel Link -->
@@ -98,5 +99,5 @@
   <mu1>1.0</mu1>
   <mu2>1.0</mu2>
-  <material>Gazebo/Yellow</material>
+  <material>Gazebo/Black</material>
 </gazebo>
 <!-- Lbwheel Link -->
@@ -132,5 +133,5 @@
   <mu1>1.0</mu1>
   <mu2>1.0</mu2>
-  <material>Gazebo/Yellow</material>
+  <material>Gazebo/Black</material>
 </gazebo>
 <!-- Rbwheel Link -->
@@ -166,5 +167,5 @@
   <mu1>1.0</mu1>
   <mu2>1.0</mu2>
-  <material>Gazebo/Yellow</material>
+  <material>Gazebo/Black</material>
 </gazebo>
 <gazebo>

File: robobase_description/models/gazebo/4differential-drive.urdf.xacro (robot description, xacro)
@@ -2,17 +2,13 @@
   <!-- Wheel separation and radius properties -->
   <!-- Wheel link names (should match those in rectangular-base) -->
-  <xacro:property name="left_front_wheel" default="lfwheel_joint"/>
-  <xacro:property name="right_front_wheel" default="rfwheel_joint"/>
   <xacro:property name="left_rear_wheel" default="lbwheel_joint"/>
   <xacro:property name="right_rear_wheel" default="rbwheel_joint"/>
   <gazebo>
     <plugin filename="gz-sim-diff-drive-system" name="gz::sim::systems::DiffDrive">
-    <num_wheel_pairs>2</num_wheel_pairs>
+    <num_wheel_pairs>1</num_wheel_pairs>
     <left_joint>lbwheel_joint</left_joint>
-    <left_joint>lfwheel_joint</left_joint>
-    <right_joint>rfwheel_joint</right_joint>
     <right_joint>rbwheel_joint</right_joint>
     <wheel_separation>0.6</wheel_separation>
-    <wheel_diameter>0.3</wheel_diameter>
+    <wheel_radius>${wheel_radius}</wheel_radius>
       <max_wheel_torque>500.0</max_wheel_torque>
       <max_linear_acceleration>5.0</max_linear_acceleration>

File: robobase_description/models/inertia_macros.xacro (robot description, xacro)
@@ -38,3 +38,21 @@
     </inertial>
   </xacro:macro>
+  <!-- Inertial for a solid sphere -->
+  <!-- If mass not provided, computed as density * (4/3) * pi * r^3 -->
+  <xacro:macro name="inertial_sphere" params="radius mass:='' density:=${default_density} *origin">
+    <xacro:if value="${mass == ''}">
+      <xacro:property name="_isphere_mass" value="${density * (4.0/3.0) * 3.141592653589793 * radius * radius * radius}"/>
+    </xacro:if>
+    <xacro:if value="${mass != ''}">
+      <xacro:property name="_isphere_mass" value="${mass}"/>
+    </xacro:if>
+    <inertial>
+      <xacro:insert_block name="origin"/>
+      <mass value="${_isphere_mass}"/>
+      <inertia
+        ixx="${(2.0/5.0) * _isphere_mass * radius * radius}" ixy="0" ixz="0"
+        iyy="${(2.0/5.0) * _isphere_mass * radius * radius}" iyz="0"
+        izz="${(2.0/5.0) * _isphere_mass * radius * radius}"/>
+    </inertial>
+  </xacro:macro>
 </robot>

File: robobase_description/models/robo.urdf.xacro (robot description, xacro)
@@ -1,9 +1,10 @@
 <?xml version="1.0"?>
 <robot xmlns:xacro="http://www.ros.org/wiki/xacro" name="robobase">
-<xacro:property name="base_length" default="0.8"/>
+<xacro:property name="base_length" default="1"/>
 <xacro:property name="base_width" default="0.45"/>
 <xacro:property name="base_height" default="0.2"/>
-<xacro:property name="wheel_radius" default="0.15"/>
-<xacro:property name="wheel_width" default="0.15"/>
+<xacro:property name="wheel_radius" default="0.2"/>
+<xacro:property name="castor_radius" default="${wheel_radius / 2}"/>
+<xacro:property name="wheel_width" default="0.2"/>
 <xacro:property name="camera_xyz" default="0.425 0 0.175"/>
 <xacro:property name="camera_rpy" default="0 0 0"/>

Commit message: hello

File: robobase_description/models/bases/rectangular-base.urdf.xacro (robot description, xacro)
@@ -63,6 +63,6 @@
     <child>lfwheel_joint</child>
   </joint>
-  <mu1>1.0</mu1>
-  <mu2>1.0</mu2>
+  <mu1>2.0</mu1>
+  <mu2>2.0</mu2>
   <material>Gazebo/Black</material>
 </gazebo>
@@ -71,17 +71,14 @@
     <parent link="base_link"/>
     <child link="rfwheel_link"/>
-    <origin xyz="${base_length / 2} -${base_width / 2} ${base_height / 2}" rpy="${pi / 2} 0 0"/>
-    <axis xyz="0 0 -1"/>
-    <limit effort="1000" velocity="1000"/>
-    <dynamics damping="1.0" friction="1.0"/>
+    <origin xyz="${base_length / 2} -${base_width / 2} 0" rpy="0 0 0"/>
 </joint>
 <link name="rfwheel_link">
-    <xacro:inertial_cylinder radius="${wheel_radius}" length="${wheel_width}">
-        <origin xyz="0 0 ${wheel_width / 2}" rpy="0 0 0"/>
-    </xacro:inertial_cylinder>
+    <xacro:inertial_sphere radius="${castor_radius}">
+        <origin xyz="0 0 0" rpy="0 0 0"/>
+    </xacro:inertial_sphere>
     <visual>
-        <origin xyz="0 0 ${wheel_width / 2}" rpy="0 0 0"/>
+        <origin xyz="0 0 0" rpy="0 0 0"/>
         <geometry>
-            <cylinder radius="${wheel_radius}" length="${wheel_width}"/>
+            <sphere radius="${castor_radius}"/>
         </geometry>
         <material name="black">
@@ -90,13 +87,17 @@
     </visual>
     <collision>
-        <origin xyz="0 0 ${wheel_width / 2}" rpy="0 0 0"/>
+        <origin xyz="0 0 0" rpy="0 0 0"/>
         <geometry>
-            <cylinder radius="${wheel_radius}" length="${wheel_width}"/>
+            <sphere radius="${castor_radius}"/>
         </geometry>
     </collision>
 </link>
 <gazebo reference="rfwheel_link">
-  <mu1>1.0</mu1>
-  <mu2>1.0</mu2>
+  <joint name="rfwheel_joint" type="ball">
+    <parent>base_link</parent>
+    <child>rfwheel_joint</child>
+  </joint>
+  <mu1>2.0</mu1>
+  <mu2>2.0</mu2>
   <material>Gazebo/Black</material>
 </gazebo>
@@ -131,6 +132,6 @@
 </link>
 <gazebo reference="lbwheel_link">
-  <mu1>1.0</mu1>
-  <mu2>1.0</mu2>
+  <mu1>2.0</mu1>
+  <mu2>2.0</mu2>
   <material>Gazebo/Black</material>
 </gazebo>
@@ -165,6 +166,6 @@
 </link>
 <gazebo reference="rbwheel_link">
-  <mu1>1.0</mu1>
-  <mu2>1.0</mu2>
+  <mu1>2.0</mu1>
+  <mu2>2.0</mu2>
   <material>Gazebo/Black</material>
 </gazebo>

File: robobase_description/models/robo.urdf.xacro (robot description, xacro)
@@ -2,14 +2,14 @@
 <robot xmlns:xacro="http://www.ros.org/wiki/xacro" name="robobase">
 <xacro:property name="base_length" default="1"/>
-<xacro:property name="base_width" default="0.45"/>
+<xacro:property name="base_width" default="0.55"/>
 <xacro:property name="base_height" default="0.2"/>
 <xacro:property name="wheel_radius" default="0.2"/>
 <xacro:property name="castor_radius" default="${wheel_radius / 2}"/>
 <xacro:property name="wheel_width" default="0.2"/>
-<xacro:property name="camera_xyz" default="0.425 0 0.175"/>
+<xacro:property name="camera_xyz" default="0.525 0 0.175"/>
 <xacro:property name="camera_rpy" default="0 0 0"/>
 <xacro:property name="camera_parent_link" default="base_link"/>
 <xacro:property name="lidar_parent_link" default="base_link"/>
-<xacro:property name="lidar_xyz" default="0 0 0.26"/>
+<xacro:property name="lidar_xyz" default="0 0 ${base_height + wheel_radius / 2}"/>
 <xacro:property name="lidar_rpy" default="0 0 0"/>
 <xacro:property name="wheel_separation" default="${base_width + wheel_width / 2}"/>

File: robobase_description/models/sensors/lidar.urdf.xacro (robot description, xacro)
@@ -12,5 +12,5 @@
       <origin xyz="0 0 0" rpy="0 0 0"/>
       <geometry>
-        <cylinder radius="0.07" length="0.12"/>
+        <cylinder radius="0.07" length="${wheel_radius}"/>
       </geometry>
       <material name="black">
@@ -19,7 +19,7 @@
     </visual>
     <collision>
-      <origin xyz="0 0 0.05" rpy="0 0 0"/>
+      <origin xyz="0 0 0" rpy="0 0 0"/>
       <geometry>
-        <cylinder radius="0.07" length="0.1"/>
+        <cylinder radius="0.07" length="${wheel_radius}"/>
       </geometry>
     </collision>

Commit message: hello

File: robobase_description/models/bases/rectangular-base.urdf.xacro (robot description, xacro)
@@ -59,10 +59,6 @@
 </link>
 <gazebo reference="lfwheel_link">
-  <joint name="lfwheel_joint" type="ball">
-    <parent>base_link</parent>
-    <child>lfwheel_joint</child>
-  </joint>
-  <mu1>2.0</mu1>
-  <mu2>2.0</mu2>
+  <mu1>3.0</mu1>
+  <mu2>3.0</mu2>
   <material>Gazebo/Black</material>
 </gazebo>
@@ -94,10 +90,6 @@
 </link>
 <gazebo reference="rfwheel_link">
-  <joint name="rfwheel_joint" type="ball">
-    <parent>base_link</parent>
-    <child>rfwheel_joint</child>
-  </joint>
-  <mu1>2.0</mu1>
-  <mu2>2.0</mu2>
+  <mu1>3.0</mu1>
+  <mu2>3.0</mu2>
   <material>Gazebo/Black</material>
 </gazebo>
@@ -132,6 +124,6 @@
 </link>
 <gazebo reference="lbwheel_link">
-  <mu1>2.0</mu1>
-  <mu2>2.0</mu2>
+  <mu1>3.0</mu1>
+  <mu2>3.0</mu2>
   <material>Gazebo/Black</material>
 </gazebo>
@@ -166,6 +158,6 @@
 </link>
 <gazebo reference="rbwheel_link">
-  <mu1>2.0</mu1>
-  <mu2>2.0</mu2>
+  <mu1>3.0</mu1>
+  <mu2>3.0</mu2>
   <material>Gazebo/Black</material>
 </gazebo>

Commit message: hello

File: robobase_description/models/bases/rectangular-base.urdf.xacro (robot description, xacro)
@@ -173,3 +173,29 @@
     </plugin>
 </gazebo>
+<gazebo>
+  <plugin filename="libgz_ros2_control-system.so" name="gz_ros2_control::GazeboSimROS2ControlPlugin">
+    <parameters>/root/robows/src/robobase/mobilerobo/config/controllers.yaml</parameters>
+  </plugin>
+</gazebo>
+<ros2_control name="GazeboSystem" type="system">
+    <hardware>
+        <plugin>gz_ros2_control/GazeboSimSystem</plugin>
+    </hardware>
+    <joint name="lbwheel_joint">
+        <command_interface name="velocity">
+        <param name="min">-10</param>
+        <param name="max">10</param>
+        </command_interface>
+        <state_interface name="position"/>
+        <state_interface name="velocity"/>
+    </joint>
+    <joint name="rbwheel_joint">
+        <command_interface name="velocity">
+        <param name="min">-10</param>
+        <param name="max">10</param>
+        </command_interface>
+        <state_interface name="position"/>
+        <state_interface name="velocity"/>
+    </joint>
+</ros2_control>
 </robot>

File: robobase_description/models/gazebo/4differential-drive.urdf.xacro (robot description, xacro)
@@ -1,2 +1,3 @@
+<?xml version="1.0"?>
 <robot xmlns:xacro="http://www.ros.org/wiki/xacro">
   <!-- Wheel separation and radius properties -->
@@ -24,5 +25,5 @@
   -->
   <!-- ROS2 Control -->
-  <ros2_control name="GazeboSystem" type="system">
+<!--   <ros2_control name="GazeboSystem" type="system">
     <hardware>
        <plugin>gz_ros2_control/GazeboSimSystem</plugin>
@@ -44,9 +45,9 @@
       <state_interface name="velocity"/>
     </joint>
-  </ros2_control>
+  </ros2_control> -->
   <!-- Gazebo ROS2 Control Plugin -->
   <gazebo>
     <plugin filename="libgz_ros2_control-system.so" name="gz_ros2_control::GazeboSimROS2ControlPlugin">
-      <parameters>$(find mobilerobo)/config/controllers.yaml</parameters>
+      <parameters>/root/robows/src/robobase/mobilerobo/config/controllers.yaml</parameters>
       <ros>
         <remapping>/tf:=tf</remapping>

File: robobase_description/models/robo.urdf.xacro (robot description, xacro)
@@ -17,4 +17,4 @@
 <xacro:include filename="$(find robobase_description)/models/sensors/camera.urdf.xacro"/>
 <xacro:include filename="$(find robobase_description)/models/sensors/lidar.urdf.xacro"/>
-<xacro:include filename="$(find robobase_description)/models/gazebo/4differential-drive.urdf.xacro"/>
+<!-- <xacro:include filename="$(find robobase_description)/models/gazebo/4differential-drive.urdf.xacro"/> -->
 </robot>

Commit message: hello

File: robobase_description/models/bases/rectangular-base.urdf.xacro (robot description, xacro)
@@ -177,4 +177,12 @@
         <plugin>gz_ros2_control/GazeboSimSystem</plugin>
     </hardware>
+    <joint name="lfwheel_joint">
+        <state_interface name="position"/>
+        <state_interface name="velocity"/>
+    </joint>
+    <joint name="rfwheel_joint">
+        <state_interface name="position"/>
+        <state_interface name="velocity"/>
+    </joint>
     <joint name="lbwheel_joint">
         <command_interface name="velocity">

File: robobase_description/models/robo.urdf.xacro (robot description, xacro)
@@ -11,5 +11,5 @@
 <xacro:property name="camera_parent_link" default="base_link"/>
 <xacro:property name="lidar_parent_link" default="base_link"/>
-<xacro:property name="lidar_xyz" default="0 0 ${base_height + wheel_radius / 2}"/>
+<xacro:property name="lidar_xyz" default="0 0 ${base_height + 0.01 + wheel_radius / 2}"/>
 <xacro:property name="lidar_rpy" default="0 0 0"/>
 <xacro:property name="wheel_separation" default="${base_width + wheel_width / 2}"/>
@@ -17,4 +17,3 @@
 <xacro:include filename="$(find robobase_description)/models/sensors/camera.urdf.xacro"/>
 <xacro:include filename="$(find robobase_description)/models/sensors/lidar.urdf.xacro"/>
-<!-- <xacro:include filename="$(find robobase_description)/models/gazebo/4differential-drive.urdf.xacro"/> -->
 </robot>

Commit message: hello

File: robobase_description/models/bases/rectangular-base.urdf.xacro (robot description, xacro)
@@ -4,5 +4,5 @@
 <xacro:include filename="$(find robobase_description)/models/inertia_macros.xacro"/>
 <link name="base_footprint">
-    <origin xyz="0 0 0" rpy="0 0 0"/>
+    <origin xyz="-${base_length / 2} 0 0" rpy="0 0 0"/>
 </link>
 <!-- Base Link -->
@@ -10,5 +10,5 @@
     <parent link="base_footprint"/>
     <child link="base_link"/>
-    <origin xyz="0 0 0" rpy="0 0 0"/>
+    <origin xyz="${base_length / 2} 0 0" rpy="0 0 0"/>
 </joint>
 <link name="base_link">

File: robobase_description/models/sensors/lidar.urdf.xacro (robot description, xacro)
@@ -47,5 +47,5 @@
           </scan>
           <range>
-            <min>0.120000</min>
+            <min>0.1</min>
             <max>8</max>
             <resolution>0.015000</resolution>

Commit message: hello

File: robobase_description/models/bases/rectangular-base.urdf.xacro (robot description, xacro)
@@ -162,10 +162,4 @@
   <material>Gazebo/Black</material>
 </gazebo>
-<!-- <gazebo>
-    <plugin name="gz::sim::systems::JointStatePublisher"
-            filename="gz-sim-joint-state-publisher-system">
-      <topic>joint_states</topic>
-    </plugin>
-</gazebo> -->
 <gazebo>
   <plugin filename="libgz_ros2_control-system.so" name="gz_ros2_control::GazeboSimROS2ControlPlugin">

File: robobase_description/models/robo.urdf.xacro (robot description, xacro)
@@ -13,7 +13,8 @@
 <xacro:property name="lidar_xyz" default="0 0 ${base_height + 0.01 + wheel_radius / 2}"/>
 <xacro:property name="lidar_rpy" default="0 0 0"/>
-<xacro:property name="wheel_separation" default="${base_width + wheel_width / 2}"/>
+<xacro:property name="wheel_separation" default="${base_width + wheel_width}"/>
 <xacro:include filename="$(find robobase_description)/models/bases/rectangular-base.urdf.xacro"/>
 <xacro:include filename="$(find robobase_description)/models/sensors/camera.urdf.xacro"/>
 <xacro:include filename="$(find robobase_description)/models/sensors/lidar.urdf.xacro"/>
+<xacro:include filename="$(find robobase_description)/models/sensors/imu.urdf.xacro"/>
 </robot>

Commit message: hello

File: robobase_description/models/bases/rectangular-base.urdf.xacro (robot description, xacro)
@@ -59,6 +59,6 @@
 </link>
 <gazebo reference="lfwheel_link">
-  <mu1>3.0</mu1>
-  <mu2>3.0</mu2>
+  <mu1>0.0</mu1>
+  <mu2>0.0</mu2>
   <material>Gazebo/Black</material>
 </gazebo>
@@ -90,6 +90,6 @@
 </link>
 <gazebo reference="rfwheel_link">
-  <mu1>3.0</mu1>
-  <mu2>3.0</mu2>
+  <mu1>0.0</mu1>
+  <mu2>0.0</mu2>
   <material>Gazebo/Black</material>
 </gazebo>

File: robobase_description/models/inertia_macros.xacro (robot description, xacro)
@@ -1,5 +1,5 @@
 <robot xmlns:xacro="http://ros.org/wiki/xacro">
   <!-- Default density (kg/m^3) -->
-  <xacro:property name="default_density" value="2700"/>
+  <xacro:property name="default_density" value="27"/>
   <!-- Inertial for a box (URDF axes aligned, origin at box center) -->
   <!-- If mass not provided, computed as density * x * y * z -->

File: robobase_description/models/sensors/imu.urdf.xacro (robot description, xacro)
@@ -10,4 +10,8 @@
 </joint>
 <link name="imu_link"/>
+<gazebo>
+    <plugin filename="gz-sim-imu-system" name="gz::sim::systems::Imu">
+    </plugin>
+</gazebo>
     <gazebo reference="imu_link">
         <sensor name="imu_sensor" type="imu">
@@ -15,4 +19,5 @@
             <update_rate>200</update_rate>
             <topic>imu</topic>
+            <gz_frame_id>imu_link</gz_frame_id>
             <imu>
             <angular_velocity>

File: robobase_description/models/temp.urdf (robot description, URDF)
Before this commit: robot robobase, 9 links, 8 joints
Joints:
- joint imu_joint: axis (none) -> 
