Commit message: hello

File: robobase_description/models/robo.urdf.xacro (robot description, xacro)
@@ -1,9 +1,12 @@
 <?xml version="1.0"?>
 <robot xmlns:xacro="http://www.ros.org/wiki/xacro" name="robobase">
-<xacro:property name="base_length" default="0.6"/>
+<xacro:property name="base_length" default="1"/>
 <xacro:property name="base_width" default="0.6"/>
 <xacro:property name="base_height" default="0.3"/>
 <xacro:property name="wheel_radius" default="0.3"/>
 <xacro:property name="wheel_width" default="0.25"/>
+<xacro:property name="camera_xyz" default="0.5 0 0.3"/>
+<xacro:property name="camera_rpy" default="0 0 0"/>
+<xacro:property name="camera_parent_link" default="base_link"/>
 <xacro:include filename="$(find robobase_description)/models/bases/rectangular-base.urdf.xacro"/>
 <xacro:include filename="$(find robobase_description)/models/sensors/camera.urdf.xacro"/>

File: robobase_description/models/sensors/camera.urdf.xacro (robot description, xacro)
@@ -1,10 +1,7 @@
 <?xml version="1.0"?>
 <robot xmlns:xacro="http://ros.org/wiki/xacro">
-  <!-- Camera pose properties (set these before including this file) -->
-  <xacro:property name="camera_xyz" default="0 0 1"/>
-  <xacro:property name="camera_rpy" default="0 0 0"/>
   <!-- Camera joint (fixed to parent, e.g., base_link) -->
   <joint name="camera_joint" type="fixed">
-    <parent link="base_link"/>
+    <parent link="${camera_parent_link}"/>
     <child link="camera_link"/>
     <origin xyz="${camera_xyz}" rpy="${camera_rpy}"/>

Commit message: hello

File: robobase_description/models/robo.urdf.xacro (robot description, xacro)
@@ -9,5 +9,9 @@
 <xacro:property name="camera_rpy" default="0 0 0"/>
 <xacro:property name="camera_parent_link" default="base_link"/>
+<xacro:property name="lidar_parent_link" default="base_link"/>
+<xacro:property name="lidar_xyz" default="0 0 0.35"/>
+<xacro:property name="lidar_rpy" default="0 0 0"/>
 <xacro:include filename="$(find robobase_description)/models/bases/rectangular-base.urdf.xacro"/>
 <xacro:include filename="$(find robobase_description)/models/sensors/camera.urdf.xacro"/>
+<xacro:include filename="$(find robobase_description)/models/sensors/lidar.urdf.xacro"/>
 </robot>

Commit message: hello

File: robobase_description/models/robo.urdf.xacro (robot description, xacro)
@@ -1,17 +1,19 @@
 <?xml version="1.0"?>
 <robot xmlns:xacro="http://www.ros.org/wiki/xacro" name="robobase">
-<xacro:property name="base_length" default="1"/>
-<xacro:property name="base_width" default="0.6"/>
-<xacro:property name="base_height" default="0.3"/>
-<xacro:property name="wheel_radius" default="0.3"/>
-<xacro:property name="wheel_width" default="0.25"/>
-<xacro:property name="camera_xyz" default="0.5 0 0.3"/>
+<xacro:property name="base_length" default="0.8"/>
+<xacro:property name="base_width" default="0.45"/>
+<xacro:property name="base_height" default="0.2"/>
+<xacro:property name="wheel_radius" default="0.15"/>
+<xacro:property name="wheel_width" default="0.15"/>
+<xacro:property name="camera_xyz" default="0.4 0 0.2"/>
 <xacro:property name="camera_rpy" default="0 0 0"/>
 <xacro:property name="camera_parent_link" default="base_link"/>
 <xacro:property name="lidar_parent_link" default="base_link"/>
-<xacro:property name="lidar_xyz" default="0 0 0.35"/>
+<xacro:property name="lidar_xyz" default="0 0 0.2"/>
 <xacro:property name="lidar_rpy" default="0 0 0"/>
+<xacro:property name="wheel_separation" default="${base_width + wheel_width / 2}"/>
 <xacro:include filename="$(find robobase_description)/models/bases/rectangular-base.urdf.xacro"/>
 <xacro:include filename="$(find robobase_description)/models/sensors/camera.urdf.xacro"/>
 <xacro:include filename="$(find robobase_description)/models/sensors/lidar.urdf.xacro"/>
+<xacro:include filename="$(find robobase_description)/models/gazebo/4differential-drive.urdf.xacro"/>
 </robot>

Commit message: hello

File: robobase_description/models/robo.urdf.xacro (robot description, xacro)
@@ -6,9 +6,9 @@
 <xacro:property name="wheel_radius" default="0.15"/>
 <xacro:property name="wheel_width" default="0.15"/>
-<xacro:property name="camera_xyz" default="0.4 0 0.2"/>
+<xacro:property name="camera_xyz" default="0.425 0 0.175"/>
 <xacro:property name="camera_rpy" default="0 0 0"/>
 <xacro:property name="camera_parent_link" default="base_link"/>
 <xacro:property name="lidar_parent_link" default="base_link"/>
-<xacro:property name="lidar_xyz" default="0 0 0.2"/>
+<xacro:property name="lidar_xyz" default="0 0 0.26"/>
 <xacro:property name="lidar_rpy" default="0 0 0"/>
 <xacro:property name="wheel_separation" default="${base_width + wheel_width / 2}"/>

File: robobase_description/models/sensors/lidar.urdf.xacro (robot description, xacro)
@@ -10,7 +10,7 @@
   <link name="lidar_link">
     <visual>
-      <origin xyz="0 0 0.05" rpy="0 0 0"/>
+      <origin xyz="0 0 0" rpy="0 0 0"/>
       <geometry>
-        <cylinder radius="0.07" length="0.1"/>
+        <cylinder radius="0.07" length="0.12"/>
       </geometry>
       <material name="black">

Commit message: hello

File: robobase_description/models/robo.urdf.xacro (robot description, xacro)
@@ -1,11 +1,11 @@
 <?xml version="1.0"?>
 <robot xmlns:xacro="http://www.ros.org/wiki/xacro" name="robobase">
-<xacro:property name="base_length" default="1"/>
-<xacro:property name="base_width" default="0.55"/>
-<xacro:property name="base_height" default="0.2"/>
-<xacro:property name="wheel_radius" default="0.2"/>
+<xacro:property name="base_length" default="0.45"/>
+<xacro:property name="base_width" default="0.32"/>
+<xacro:property name="base_height" default="0.1"/>
+<xacro:property name="wheel_radius" default="0.1"/>
 <xacro:property name="castor_radius" default="${wheel_radius / 2}"/>
-<xacro:property name="wheel_width" default="0.2"/>
-<xacro:property name="camera_xyz" default="0.525 0 0.175"/>
+<xacro:property name="wheel_width" default="0.06"/>
+<xacro:property name="camera_xyz" default="${base_length / 2 + 0.001} 0 ${base_height / 2 + 0.001}"/>
 <xacro:property name="camera_rpy" default="0 0 0"/>
 <xacro:property name="camera_parent_link" default="base_link"/>

File: robobase_description/models/sensors/camera.urdf.xacro (robot description, xacro)
@@ -11,5 +11,5 @@
     <visual>
       <geometry>
-        <box size="0.05 0.05 0.05"/>
+        <box size="0.02 0.02 0.02"/>
       </geometry>
       <material name="black"/>
@@ -17,5 +17,5 @@
     <collision>
       <geometry>
-        <box size="0.05 0.05 0.05"/>
+        <box size="0.02 0.02 0.02"/>
       </geometry>
     </collision>

File: robobase_description/models/sensors/lidar.urdf.xacro (robot description, xacro)
@@ -12,5 +12,5 @@
       <origin xyz="0 0 0" rpy="0 0 0"/>
       <geometry>
-        <cylinder radius="0.07" length="${wheel_radius}"/>
+        <cylinder radius="0.03" length="${wheel_radius}"/>
       </geometry>
       <material name="black">
@@ -21,10 +21,10 @@
       <origin xyz="0 0 0" rpy="0 0 0"/>
       <geometry>
-        <cylinder radius="0.07" length="${wheel_radius}"/>
+        <cylinder radius="0.03" length="${wheel_radius}"/>
       </geometry>
     </collision>
     <inertial>
       <mass value="0.5"/>
-      <origin xyz="0 0 0.05" rpy="0 0 0"/>
+      <origin xyz="0 0 0" rpy="0 0 0"/>
       <inertia ixx="0.001" ixy="0" ixz="0" iyy="0.001" iyz="0" izz="0.001"/>
     </inertial>
